Commit message: franka_description/CMakeLists.txt

File: robot_models/franka_description/robots/panda.gazebo.xacro (robot description, xacro)
@@ -63,3 +63,42 @@
         </gazebo>
     </xacro:macro>
+<gazebo reference="camera_link">
+    <sensor type="camera" name="camera1">
+      <update_rate>30.0</update_rate>
+      <camera name="head">
+        <horizontal_fov>1.3962634</horizontal_fov>
+        <image>
+          <width>800</width>
+          <height>800</height>
+          <format>R8G8B8</format>
+        </image>
+        <clip>
+          <near>0.02</near>
+          <far>300</far>
+        </clip>
+        <noise>
+          <type>gaussian</type>
+          <!-- Noise is sampled independently per pixel on each frame.
+               That pixel's noise value is added to each of its color
+               channels, which at that point lie in the range [0,1]. -->
+          <mean>0.0</mean>
+          <stddev>0.007</stddev>
+        </noise>
+      </camera>
+      <plugin name="camera_controller" filename="libgazebo_ros_camera.so">
+        <alwaysOn>true</alwaysOn>
+        <updateRate>0.0</updateRate>
+        <cameraName>rrbot/camera1</cameraName>
+        <imageTopicName>image_raw</imageTopicName>
+        <cameraInfoTopicName>camera_info</cameraInfoTopicName>
+        <frameName>camera_link</frameName>
+        <hackBaseline>0.07</hackBaseline>
+        <distortionK1>0.0</distortionK1>
+        <distortionK2>0.0</distortionK2>
+        <distortionK3>0.0</distortionK3>
+        <distortionT1>0.0</distortionT1>
+        <distortionT2>0.0</distortionT2>
+      </plugin>
+    </sensor>
+  </gazebo>
 </robot>

File: robot_models/franka_description/robots/panda.transmission.xacro (robot description, xacro)
@@ -11,5 +11,5 @@
         <transmission name="${robot_name}_tran_1">
             <type>transmission_interface/SimpleTransmission</type>
-            <joint name="${robot_name}_joint1">
+            <joint name="joint1">
                 <hardwareInterface>hardware_interface/EffortJointInterface</hardwareInterface>
             </joint>
@@ -21,5 +21,5 @@
         <transmission name="${robot_name}_tran_2">
             <type>transmission_interface/SimpleTransmission</type>
-            <joint name="${robot_name}_joint2">
+            <joint name="joint2">
                 <hardwareInterface>hardware_interface/EffortJointInterface</hardwareInterface>
             </joint>
@@ -31,5 +31,5 @@
         <transmission name="${robot_name}_tran_3">
             <type>transmission_interface/SimpleTransmission</type>
-            <joint name="${robot_name}_joint3">
+            <joint name="joint3">
                 <hardwareInterface>hardware_interface/EffortJointInterface</hardwareInterface>
             </joint>
@@ -41,5 +41,5 @@
         <transmission name="${robot_name}_tran_4">
             <type>transmission_interface/SimpleTransmission</type>
-            <joint name="${robot_name}_joint4">
+            <joint name="joint4">
                 <hardwareInterface>hardware_interface/EffortJointInterface</hardwareInterface>
             </joint>
@@ -51,5 +51,5 @@
         <transmission name="${robot_name}_tran_5">
             <type>transmission_interface/SimpleTransmission</type>
-            <joint name="${robot_name}_joint5">
+            <joint name="joint5">
                 <hardwareInterface>hardware_interface/EffortJointInterface</hardwareInterface>
             </joint>
@@ -61,5 +61,5 @@
         <transmission name="${robot_name}_tran_6">
             <type>transmission_interface/SimpleTransmission</type>
-            <joint name="${robot_name}_joint6">
+            <joint name="joint6">
                 <hardwareInterface>hardware_interface/EffortJointInterface</hardwareInterface>
             </joint>
@@ -71,5 +71,5 @@
         <transmission name="${robot_name}_tran_7">
             <type>transmission_interface/SimpleTransmission</type>
-            <joint name="${robot_name}_joint7">
+            <joint name="joint7">
                 <hardwareInterface>hardware_interface/EffortJointInterface</hardwareInterface>
             </joint>

File: robot_models/franka_description/robots/panda_arm.xacro (robot description, xacro)
@@ -3,5 +3,5 @@
   <xacro:macro name="panda_arm" params="arm_id:='panda' description_pkg:='franka_description' connected_to:='' xyz:='0 0 0' rpy:='0 0 0'">
     <xacro:unless value="${not connected_to}">
-      <joint name="${arm_id}_joint_${connected_to}" type="fixed">
+      <joint name="joint_${connected_to}" type="fixed">
         <parent link="${connected_to}"/>
         <child link="${arm_id}_link0"/>
@@ -50,5 +50,5 @@
       <!-- end for simulation -->
     </link>
-    <joint name="${arm_id}_joint1" type="revolute">
+    <joint name="joint1" type="revolute">
       <safety_controller k_position="100.0" k_velocity="40.0" soft_lower_limit="-2.8973" soft_upper_limit="2.8973"/>
       <origin rpy="0 0 0" xyz="0 0 0.333"/>
@@ -80,5 +80,5 @@
       <!-- end for simulation -->
     </link>
-    <joint name="${arm_id}_joint2" type="revolute">
+    <joint name="joint2" type="revolute">
       <safety_controller k_position="100.0" k_velocity="40.0" soft_lower_limit="-1.7628" soft_upper_limit="1.7628"/>
       <origin rpy="${-pi/2} 0 0" xyz="0 0 0"/>
@@ -110,5 +110,5 @@
       <!-- end for simulation -->
     </link>
-    <joint name="${arm_id}_joint3" type="revolute">
+    <joint name="joint3" type="revolute">
       <safety_controller k_position="100.0" k_velocity="40.0" soft_lower_limit="-2.8973" soft_upper_limit="2.8973"/>
       <origin rpy="${pi/2} 0 0" xyz="0 -0.316 0"/>
@@ -140,5 +140,5 @@
       <!-- end for simulation -->
     </link>
-    <joint name="${arm_id}_joint4" type="revolute">
+    <joint name="joint4" type="revolute">
       <safety_controller k_position="100.0" k_velocity="40.0" soft_lower_limit="-3.0718" soft_upper_limit="-0.0698"/>
       <origin rpy="${pi/2} 0 0" xyz="0.0825 0 0"/>
@@ -170,5 +170,5 @@
       <!-- end for simulation -->
     </link>
-    <joint name="${arm_id}_joint5" type="revolute">
+    <joint name="joint5" type="revolute">
       <safety_controller k_position="100.0" k_velocity="40.0" soft_lower_limit="-2.8973" soft_upper_limit="2.8973"/>
       <origin rpy="${-pi/2} 0 0" xyz="-0.0825 0.384 0"/>
@@ -200,5 +200,5 @@
       <!-- end for simulation -->
     </link>
-    <joint name="${arm_id}_joint6" type="revolute">
+    <joint name="joint6" type="revolute">
       <safety_controller k_position="100.0" k_velocity="40.0" soft_lower_limit="-0.0175" soft_upper_limit="3.7525"/>
       <origin rpy="${pi/2} 0 0" xyz="0 0 0"/>
@@ -230,5 +230,5 @@
       <!-- end for simulation -->
     </link>
-    <joint name="${arm_id}_joint7" type="revolute">
+    <joint name="joint7" type="revolute">
       <safety_controller k_position="100.0" k_velocity="40.0" soft_lower_limit="-2.8973" soft_upper_limit="2.8973"/>
       <origin rpy="${pi/2} 0 0" xyz="0.088 0 0"/>
@@ -236,5 +236,5 @@
       <child link="${arm_id}_link7"/>
       <axis xyz="0 0 1"/>
-      <limit effort="12" lower="-2.8973" upper="2.8973" velocity="2.6100"/>
+      <limit effort="12" lower="-2.8973" upper="2.8973" velocity="2.6100s"/>
       <!-- for simulation -->
       <dynamics damping="${joint_damping}" friction="0.5649"/>
@@ -250,5 +250,5 @@
       <!-- end for simulation -->
     </link>
-    <joint name="${arm_id}_joint8" type="fixed">
+    <joint name="joint8" type="fixed">
       <origin rpy="0 0 0" xyz="0 0 0.107"/>
       <parent link="${arm_id}_link7"/>
@@ -256,4 +256,32 @@
       <axis xyz="0 0 0"/>
     </joint>
+<joint name="camera_joint" type="fixed">
+   <axis xyz="0 1 0" />
+   <origin xyz="0 0 0.05" rpy="${3.1415} ${-3.1415/2} 0"/>
+   <parent link="${arm_id}_link8"/>
+   <child link="camera_link"/>
+ </joint>
+<xacro:property name="camera_side" value="0.05" />
+ <!-- Camera -->
+ <link name="camera_link">
+   <collision>
+     <origin xyz="0 0 0" rpy="0 0 0"/>
+     <geometry>
+   <box size="${camera_side} ${camera_side} ${camera_side}"/>
+     </geometry>
+   </collision>
+   <visual>
+     <origin xyz="0 0 0" rpy="0 0 0"/>
+     <geometry>
+   <box size="${camera_side} ${camera_side} ${camera_side}"/>
+     </geometry>
+     <material name="red"/>
+   </visual>
+   <inertial>
+     <mass value="1e-5" />
+     <origin xyz="0 0 0" rpy="0 0 0"/>
+     <inertia ixx="1e-6" ixy="0" ixz="0" iyy="1e-6" iyz="0" izz="1e-6" />
+   </inertial>
+ </link>
   </xacro:macro>
 </robot>
